File: BT_Keyboard/BT_Keyboard.kicad_pcb (KiCad board)
At the start: 2 copper layers, 285.9 x 114.5 mm, 154 parts, among them SW1 SW_Push_45deg, SW10 SW_Push_45deg, SW11 SW_Push_45deg, SW12 SW_Push_45deg, SW13 SW_Push_45deg, SW14 SW_Push_45deg, SW15 SW_Push_45deg, SW16 SW_Push_45deg, SW17 SW_Push_45deg, SW18 SW_Push_45deg, SW19 SW_Push_45deg, SW2 SW_Push_45deg, SW20 SW_Push_45deg, SW21 SW_Push_45deg, SW22 SW_Push_45deg, SW23 SW_Push_45deg, SW24 SW_Push_45deg, SW25 SW_Push_45deg, SW26 SW_Push_45deg, SW27 SW_Push_45deg, SW28 Backspace, SW29 Tab, SW3 SW_Push_45deg, SW30 Cap, SW31 SW_Push_45deg, SW32 SW_Push_45deg, SW33 SW_Push_45deg, SW34 SW_Push_45deg, SW35 SW_Push_45deg, SW36 SW_Push_45deg, SW37 SW_Push_45deg, SW38 SW_Push_45deg, SW39 SW_Push_45deg, SW4 SW_Push_45deg, SW40 SW_Push_45deg, SW41 SW_Push_45deg, SW42 SW_Push_45deg, SW43 SW_Push_45deg, SW44 SW_Push_45deg, SW45 SW_Push_45deg, SW46 SW_Push_45deg, SW47 SW_Push_45deg, SW48 SW_Push_45deg, SW49 SW_Push_45deg, SW5 SW_Push_45deg, SW50 SW_Push_45deg, SW51 SW_Push_45deg, SW52 SW_Push_45deg, SW53 SW_Push_45deg, SW54 Enter, SW55 SW_Push_45deg, SW56 Shift, SW57 SW_Push_45deg, SW58 SW_Push_45deg, SW59 SW_Push_45deg, SW6 SW_Push_45deg, SW60 SW_Push_45deg, SW61 SW_Push_45deg, SW62 SW_Push_45deg, SW63 SW_Push_45deg, SW64 SW_Push_45deg, SW65 SW_Push_45deg, SW66 SW_Push_45deg, SW67 SW_Push_45deg, SW68 SW_Push_45deg, SW69 SW_Push_45deg, SW7 SW_Push_45deg, SW70 SW_Push_45deg, SW71 SW_Push_45deg, SW72 SW_Push_45deg, SW73 SW_Push_45deg, SW74 SW_Push_45deg, SW75 SW_Push_45deg, SW76 SW_Push_45deg, SW77 SW_Push_45deg, SW8 SW_Push_45deg, SW9 SW_Push_45deg

Commit message: Add files via upload
Parts:
- added D80: LED, LED_THT:LED_D5.0mm, F.Cu at (171.3, 101.4)
- added D81: LED, LED_THT:LED_D5.0mm, F.Cu at (180.2, 101.4)
- added J1: Conn_01x22_Pin, Connector_PinHeader_2.54mm:PinHeader_1x22_P2.54mm_Vertical, F.Cu at (225.3, 123.6)
- added J2: Conn_01x22_Pin, Connector_PinHeader_2.54mm:PinHeader_1x22_P2.54mm_Vertical, F.Cu at (225.3, 97.1)
- added J3: Conn_01x14_Pin, Connector_PinHeader_2.54mm:PinHeader_1x14_P2.54mm_Vertical, F.Cu at (173.5, 81.6)
- added J4: Conn_01x22_Pin, Connector_PinHeader_2.54mm:PinHeader_1x22_P2.54mm_Vertical, F.Cu at (225.3, 100.7)
- added J5: Conn_01x22_Pin, Connector_PinHeader_2.54mm:PinHeader_1x22_P2.54mm_Vertical, F.Cu at (225.3, 127.2)
- SW30: value Cap -> SW_Push_45deg; footprint Button_Switch_Keyboard:SW_Cherry_MX_1.50u_PCB -> Button_Switch_Keyboard:SW_Cherry_MX_1.00u_PCB
- SW43: value SW_Push_45deg -> Cap; footprint Button_Switch_Keyboard:SW_Cherry_MX_1.00u_PCB -> Button_Switch_Keyboard:SW_Cherry_MX_1.50u_PCB
- SW54: value Enter -> SW_Push_45deg; footprint Button_Switch_Keyboard:SW_Cherry_MX_2.00u_PCB -> Button_Switch_Keyboard:SW_Cherry_MX_1.00u_PCB
- SW55: value SW_Push_45deg -> Enter; footprint Button_Switch_Keyboard:SW_Cherry_MX_1.00u_PCB -> Button_Switch_Keyboard:SW_Cherry_MX_2.00u_PCB
- moved SW11 127.9 mm to (356.5, 37.6)
- moved SW25 127.9 mm to (356.5, 56.6)
- moved SW51 127.9 mm to (332.7, 94.7)
- moved SW66 127.9 mm to (380.3, 113.8)
- moved SW73 127.9 mm to (356.5, 132.8)
- moved SW10 127.9 mm to (337.5, 37.6)
- moved SW13 127.9 mm to (394.6, 37.6)
- moved SW14 127.9 mm to (432.7, 37.6)
- moved SW23 127.9 mm to (318.4, 56.6)
- moved SW24 127.9 mm to (337.5, 56.6)
- moved SW27 127.9 mm to (394.6, 56.6)
- moved SW28 127.9 mm to (423.2, 56.6)
- moved SW38 127.9 mm to (347.0, 75.7)
- moved SW39 127.9 mm to (366.1, 75.7)
- moved SW40 127.9 mm to (385.1, 75.7)
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Connections:
- D30 pad 1: X0 -> X1
- D31 pad 1: X1 -> X2
- D32 pad 1: X1 -> X3
- D33 pad 1: X2 -> X4
- D34 pad 1: X2 -> X5
- D35 pad 1: X3 -> X6
- D36 pad 1: X3 -> X7
- D37 pad 1: X4 -> X8
- D38 pad 1: X4 -> X9
- D39 pad 1: X5 -> X10
- D40 pad 1: X5 -> X11
- D41 pad 1: X6 -> X12
- D42 pad 1: X6 -> X13
- D43 pad 1: X7 -> X0
- D44 pad 1: X7 -> X1
- D45 pad 1: X8 -> X2
- D46 pad 1: X8 -> X3
- D47 pad 1: X9 -> X4
- D48 pad 1: X9 -> X5
- D49 pad 1: X10 -> X6
- D50 pad 1: X10 -> X7
- D51 pad 1: X11 -> X8
- D52 pad 1: X11 -> X9
- D53 pad 1: X12 -> X10
- D54 pad 1: X12 -> X11
- D55 pad 1: X13 -> X12
- SW30 pad 1: Y3 -> Y2
- SW32 pad 1: Y3 -> Y2
- SW34 pad 1: Y3 -> Y2
- SW36 pad 1: Y3 -> Y2
- SW38 pad 1: Y3 -> Y2
- SW40 pad 1: Y3 -> Y2
- SW42 pad 1: Y3 -> Y2
- SW43 pad 1: Y2 -> Y3
- SW45 pad 1: Y2 -> Y3
- SW47 pad 1: Y2 -> Y3
- SW49 pad 1: Y2 -> Y3
- SW51 pad 1: Y2 -> Y3
- SW53 pad 1: Y2 -> Y3
- SW55 pad 1: Y2 -> Y3
Routing:
- net Y5: track 279.5 -> 564.7 mm
- net X13: track 62.1 -> 290.7 mm
- net Y0: track 288.5 -> 508.4 mm, vias 0 -> 2
- net X0: track 129.1 -> 340.4 mm
- net Y1: track 275.6 -> 485.0 mm, vias 0 -> 2
- net X12: track 80.6 -> 284.7 mm
- net Y4: track 253.5 -> 445.6 mm
- net RESET: track 0.00 -> 184.1 mm
- net X1: track 145.5 -> 325.3 mm
- net GND: track 0.00 -> 151.8 mm, vias 0 -> 1
- net X6: track 259.5 -> 409.7 mm, vias 1 -> 0
- net SCK: track 0.00 -> 148.6 mm
- net SDO: track 0.00 -> 137.0 mm
- net X2: track 168.5 -> 300.4 mm, vias 1 -> 0
- net SDI: track 0.00 -> 131.8 mm
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Other:
- board size 285.9 x 114.5 mm -> 414.8 x 114.4 mm
- board text added: "ESC F1 F2 F3 F4 F5 F6 F7 F8 F9 F10 F11 F12 Del ` 1 2 3 4 5 6 7 8 9 0 - = BackSpace Tab q w e r t y u i o p [ ] \ Caps a s d f g h j k l ; ' Enter Shift z x c v b n m , . / Up Ctrl Fn Windows Alt Space Alt Ctrl left Down right"
- board text added: "Retro-Pad"

Commit message: Add files via upload
Parts:
- added J7: Speaker, Connector_PinSocket_2.54mm:PinSocket_1x02_P2.54mm_Vertical, F.Cu at (192.0, 97.3)
- added J8: Battery 5V, Connector_PinSocket_2.54mm:PinSocket_1x02_P2.54mm_Vertical, F.Cu at (181.3, 108.1)
Connections:
- net Net-(J2-Pin_4) renamed Speaker
- net Net-(J2-Pin_5) renamed Resis_Strip
Routing:
- net 5V: track 112.6 -> 210.5 mm
- net Speaker: track 3.60 -> 48.1 mm
- net GND: track 151.8 -> 169.9 mm

Commit message: Add files via upload
Parts:
- SW1, SW10, SW11, SW12, SW13, SW14, SW15, SW16, SW17, SW18, SW19, SW2, SW20, SW21, SW22, SW23, SW24, SW25, SW26, SW27, SW3, SW30, SW31, SW32, SW33, SW34, SW35, SW36, SW37, SW38, SW39, SW4, SW40, SW41, SW42, SW44, SW45, SW46, SW47, SW48, SW49, SW5, SW50, SW51, SW52, SW53, SW54, SW57, SW58, SW59, SW6, SW60, SW61, SW62, SW63, SW64, SW65, SW66, SW67, SW68, SW69, SW7, SW70, SW71, SW72, SW73, SW74, SW75, SW76, SW77, SW8, SW9: footprint Button_Switch_Keyboard:SW_Cherry_MX_1.00u_PCB -> PCM_Switch_Keyboard_Hotswap_Kailh:SW_Hotswap_Kailh_MX_Plated_1.00u
- SW28: footprint Button_Switch_Keyboard:SW_Cherry_MX_1.75u_PCB -> PCM_Switch_Keyboard_Hotswap_Kailh:SW_Hotswap_Kailh_MX_Plated_1.75u
- SW29: footprint Button_Switch_Keyboard:SW_Cherry_MX_1.25u_PCB -> PCM_Switch_Keyboard_Hotswap_Kailh:SW_Hotswap_Kailh_MX_Plated_1.25u
- SW43: footprint Button_Switch_Keyboard:SW_Cherry_MX_1.50u_PCB -> PCM_Switch_Keyboard_Hotswap_Kailh:SW_Hotswap_Kailh_MX_Plated_1.50u
- SW55, SW56: footprint Button_Switch_Keyboard:SW_Cherry_MX_2.00u_PCB -> PCM_Switch_Keyboard_Hotswap_Kailh:SW_Hotswap_Kailh_MX_Plated_2.00u
- moved SW65 5.89 mm to (358.2, 118.8)
- moved SW66 5.89 mm to (377.3, 118.8)
- moved SW73 5.89 mm to (353.4, 137.8)
- moved SW77 5.89 mm to (429.6, 137.8)
- moved SW10 5.89 mm to (334.4, 42.6)
- moved SW11 5.89 mm to (353.4, 42.6)
- moved SW14 5.89 mm to (429.6, 42.6)
- moved SW22 5.89 mm to (296.2, 61.6)
- moved SW24 5.89 mm to (334.4, 61.6)
- moved SW25 5.89 mm to (353.4, 61.6)
- moved SW8 5.89 mm to (296.2, 42.6)
- moved SW36 5.89 mm to (305.8, 80.7)
- moved SW40 5.89 mm to (382.0, 80.7)
- moved SW41 5.89 mm to (401.1, 80.7)
- moved SW42 5.89 mm to (424.9, 80.7)
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Connections:
- net Resis_Strip renamed Net-(J2-Pin_5)
Routing:
- net RESET: track 184.1 -> 83.6 mm
- net Y5: track 564.7 -> 479.5 mm, vias 0 -> 1
- net 5V: track 210.5 -> 152.5 mm
- net SCK: track 148.6 -> 112.5 mm
- net X10: track 234.5 -> 269.0 mm
- net Y2: track 485.8 -> 519.3 mm, vias 2 -> 1
- net Y0: track 508.4 -> 541.4 mm, vias 2 -> 3
- net X4: track 253.2 -> 220.8 mm
- net FN: track 107.2 -> 138.2 mm
- net X11: track 279.8 -> 310.5 mm
- net Y1: track 485.0 -> 514.7 mm, vias 2 -> 3
- net X13: track 290.7 -> 317.5 mm
- net GND: track 169.9 -> 144.4 mm, vias 1 -> 0
- net SDI: track 131.8 -> 107.7 mm
- net SDO: track 137.0 -> 115.9 mm
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Other:
- board size 414.8 x 114.4 mm -> 414.8 x 120.7 mm

Commit message: Add files via upload
Parts:
- moved SW72 0.11 mm to (166.7, 137.8)
Changed lines of the file:
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@@
 	(footprint "PCM_Switch_Keyboard_Hotswap_Kailh:SW_Hotswap_Kailh_MX_Plated_1.00u"
 		(layer "F.Cu")
-		(at 166.60125 137.84)
+		(at 166.7 137.8)
 		(descr "Kailh keyswitch Hotswap Socket plated holes Keycap 1.00u")
 		(tags "Kailh Keyboard Keyswitch Switch Hotswap Socket Plated Relief Cutout Keycap 1.00u")
@@
 	)
 	(segment
-		(start 125.8 136.20375)
-		(end 113.89375 148.11)
-		(width 0.2)
-		(layer "F.Cu")
-		(net "X3")
-	)
-	(segment
 		(start 111.5125 86.571598)
 		(end 111.5125 90.96)
@@
 	(segment
 		(start 125.8 129.06)
-		(end 125.8 136.20375)
+		(end 121.1 133.76)
+		(width 0.2)
+		(layer "F.Cu")
+		(net "X3")
+	)
+	(segment
+		(start 121.1 133.76)
+		(end 121.1 140.90375)
+		(width 0.2)
+		(layer "F.Cu")
+		(net "X3")
+	)
+	(segment
+		(start 121.1 140.90375)
+		(end 113.89375 148.11)
 		(width 0.2)
 		(layer "F.Cu")
@@
 	)
 	(segment
+		(start 235.426179 97.1)
+		(end 235.426179 100.7)
+		(width 0.2)
+		(layer "B.Cu")
+		(net "Net-(J2-Pin_5)")
+	)
+	(segment
 		(start 253.206179 97.1)
 		(end 253.206179 100.7)
@@
 		(net "Net-(D64-A)")
 	)
-	(segment
-		(start 235.426179 97.1)
-		(end 235.426179 100.7)
-		(width 0.2)
-		(layer "B.Cu")
-		(net "Net-(J2-Pin_5)")
-	)
 	(embedded_fonts no)
