File: BT_Keyboard/BT_Keyboard.kicad_pcb (KiCad board)
At the start: 2 copper layers, 414.8 x 120.7 mm, 163 parts, among them J1 Conn_01x22_Pin, J2 Conn_01x22_Pin, J3 Conn_01x14_Pin, J4 Conn_01x22_Pin, J5 Conn_01x22_Pin, J7 Speaker, J8 Battery 5V, SW1 SW_Push_45deg, SW10 SW_Push_45deg, SW11 SW_Push_45deg, SW12 SW_Push_45deg, SW13 SW_Push_45deg, SW14 SW_Push_45deg, SW15 SW_Push_45deg, SW16 SW_Push_45deg, SW17 SW_Push_45deg, SW18 SW_Push_45deg, SW19 SW_Push_45deg, SW2 SW_Push_45deg, SW20 SW_Push_45deg, SW21 SW_Push_45deg, SW22 SW_Push_45deg, SW23 SW_Push_45deg, SW24 SW_Push_45deg, SW25 SW_Push_45deg, SW26 SW_Push_45deg, SW27 SW_Push_45deg, SW28 Backspace, SW29 Tab, SW3 SW_Push_45deg, SW30 SW_Push_45deg, SW31 SW_Push_45deg, SW32 SW_Push_45deg, SW33 SW_Push_45deg, SW34 SW_Push_45deg, SW35 SW_Push_45deg, SW36 SW_Push_45deg, SW37 SW_Push_45deg, SW38 SW_Push_45deg, SW39 SW_Push_45deg, SW4 SW_Push_45deg, SW40 SW_Push_45deg, SW41 SW_Push_45deg, SW42 SW_Push_45deg, SW43 Cap, SW44 SW_Push_45deg, SW45 SW_Push_45deg, SW46 SW_Push_45deg, SW47 SW_Push_45deg, SW48 SW_Push_45deg, SW49 SW_Push_45deg, SW5 SW_Push_45deg, SW50 SW_Push_45deg, SW51 SW_Push_45deg, SW52 SW_Push_45deg, SW53 SW_Push_45deg, SW54 SW_Push_45deg, SW55 Enter, SW56 Shift, SW57 SW_Push_45deg, SW58 SW_Push_45deg, SW59 SW_Push_45deg, SW6 SW_Push_45deg, SW60 SW_Push_45deg, SW61 SW_Push_45deg, SW62 SW_Push_45deg, SW63 SW_Push_45deg, SW64 SW_Push_45deg, SW65 SW_Push_45deg, SW66 SW_Push_45deg, SW67 SW_Push_45deg, SW68 SW_Push_45deg, SW69 SW_Push_45deg, SW7 SW_Push_45deg, SW70 SW_Push_45deg, SW71 SW_Push_45deg, SW72 SW_Push_45deg, SW73 SW_Push_45deg, SW74 SW_Push_45deg, SW75 SW_Push_45deg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

Commit message: Add files via upload
Parts:
- removed J1, J2: Conn_01x22_Pin, Connector_PinHeader_2.54mm:PinHeader_1x22_P2.54mm_Vertical
- moved J4 52.7 mm to (278.0, 100.6), turned to -90 degrees
- moved J3 33.0 mm to (173.5, 48.5), turned to 0 degrees
- moved J8 4.53 mm to (181.3, 112.7)
- moved J7 3.50 mm to (192.0, 100.8)
- moved J5 1.37 mm to (224.6, 126.0)
Connections:
- J4 pad 10: Y4 -> X11
- J4 pad 11: Y5 -> X12
- J4 pad 12: Net-(J2-Pin_12) -> Y3
- J4 pad 13: Net-(J2-Pin_13) -> Y1
- J4 pad 14: Net-(J2-Pin_14) -> X8
- J4 pad 20: Net-(J2-Pin_20) -> RESET
- J4 pad 4: Speaker -> X4
- J4 pad 5: Net-(J2-Pin_5) -> X5
- J4 pad 6: Y0 -> X6
- J4 pad 7: Y1 -> X7
- J4 pad 8: Y2 -> X9
- J4 pad 9: Y3 -> X10
- J5 pad 10: X8 -> Net-(J1-Pin_10)
- J5 pad 11: X7 -> Net-(J1-Pin_11)
- J5 pad 12: X6 -> Net-(J1-Pin_12)
- J5 pad 13: X5 -> X0
- J5 pad 14: X4 -> X1
- J5 pad 15: X3 -> X2
- J5 pad 16: X2 -> X3
- J5 pad 17: X1 -> Y5
- J5 pad 18: X0 -> FN
- J5 pad 19: Net-(J1-Pin_19) -> NUM
- J5 pad 20: FN -> Net-(J1-Pin_20)
- J5 pad 21: NUM -> Speaker
- J5 pad 4: RESET -> Net-(J1-Pin_4)
- J5 pad 5: X13 -> LED
- J5 pad 6: X12 -> X13
- J5 pad 7: X11 -> Y0
- J5 pad 8: X10 -> Y2
- J5 pad 9: X9 -> Y4
Routing:
- net LED: track 0.00 -> 114.3 mm
- net X9: track 377.1 -> 282.2 mm, vias 0 -> 1
- net X7: track 331.7 -> 238.0 mm, vias 0 -> 1
- net X5: track 302.7 -> 396.4 mm, vias 0 -> 1
- net X8: track 356.9 -> 283.2 mm, vias 0 -> 1
- net Speaker: track 49.4 -> 108.0 mm, vias 0 -> 1
- net X12: track 303.6 -> 258.5 mm, vias 0 -> 1
- net X4: track 220.8 -> 263.4 mm, vias 0 -> 2
- net X11: track 310.5 -> 271.9 mm, vias 0 -> 1
- net X6: track 400.8 -> 363.7 mm, vias 0 -> 1
- net FN: track 138.2 -> 103.2 mm, vias 0 -> 1
- net Y5: track 479.5 -> 444.6 mm
- net SDO: track 115.9 -> 84.4 mm, vias 0 -> 1
- net RESET: track 83.6 -> 113.8 mm
- net X10: track 269.0 -> 240.6 mm, vias 0 -> 1
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Other:
- board text removed: "Retro-Pad"
